Commit message: ✨ feat(add d435i to scoutv2):

File: src/scout_simulator/scout_description/urdf/scout_v2.xacro (robot description, xacro)
@@ -1,15 +1,19 @@
 <?xml version="1.0"?>
-<robot name="scout_v2"
-    xmlns:xacro="http://ros.org/wiki/xacro">
+<robot name="scout_v2" xmlns:xacro="http://ros.org/wiki/xacro">
     <xacro:arg name="robot_namespace" default="/" />
     <xacro:arg name="urdf_extras" default="empty.urdf" />
     <xacro:include filename="$(find scout_description)/urdf/scout_wheel_type1.xacro" />
     <xacro:include filename="$(find scout_description)/urdf/scout_wheel_type2.xacro" />
-    <xacro:include filename="$(find velodyne_description)/urdf/HDL-32E.urdf.xacro"/>
+    <xacro:include filename="$(find velodyne_description)/urdf/HDL-32E.urdf.xacro" />
     <xacro:HDL-32E parent="base_link" name="velodyne" topic="/velodyne_points" hz="10" samples="440" gpu="false" lasers="32" max_range="100">
         <origin xyz="0 0 0.3" rpy="0 0 0" />
     </xacro:HDL-32E>
+    <!-- d435i frame definition can be found at https://github.com/IntelRealSense/librealsense/blob/master/doc/d435i.md -->
+    <xacro:include filename="$(find realsense_gazebo_description)/urdf/_d435i.urdf.xacro" />
+    <xacro:sensor_d435i parent="base_link" name="D435i_camera" topics_ns="D435i_camera">
+        <origin xyz="0.05 0 0.3" rpy="0 0 0 " />
+    </xacro:sensor_d435i>
     <!-- Variables -->
-    <xacro:property name="M_PI" value="3.14159"/>
+    <xacro:property name="M_PI" value="3.14159" />
     <!-- Vehicle Geometries -->
     <xacro:property name="base_x_size" value="0.9250000" />
@@ -32,5 +36,5 @@
             <origin xyz="0 0 0.008" rpy="0 0 0" />
             <geometry>
-                <box size="${base_x_size} ${base_y_size} ${base_z_size}"/>
+                <box size="${base_x_size} ${base_y_size} ${base_z_size}" />
             </geometry>
         </collision>
@@ -38,5 +42,5 @@
             <origin xyz="0 0 ${base_z_size/6}" rpy="0 0 0" />
             <geometry>
-                <box size="${base_x_size/6} ${base_y_size*1.65} ${base_z_size/3}"/>
+                <box size="${base_x_size/6} ${base_y_size*1.65} ${base_z_size/3}" />
             </geometry>
         </collision>
