Commit message: ✨ feat(enable LVI-SAM):

File: src/scout_simulator/scout_description/urdf/scout_v2_cam_imu.xacro (robot description, xacro)
@@ -7,6 +7,11 @@
     <xacro:include filename="$(find velodyne_description)/urdf/HDL-32E.urdf.xacro" />
     <xacro:HDL-32E parent="base_link" name="velodyne" topic="/velodyne_points" hz="10" samples="440" gpu="false" lasers="32" max_range="100">
-        <origin xyz="0 0 0.3" rpy="0 0 0" />
+        <origin xyz="0 0 0.6" rpy="0 0 0" />
     </xacro:HDL-32E>
+    <!-- d435i frame definition can be found at https://github.com/IntelRealSense/librealsense/blob/master/doc/d435i.md -->
+    <!-- <xacro:include filename="$(find realsense_gazebo_description)/urdf/_d435i.urdf.xacro" />
+    <xacro:sensor_d435i parent="base_link" name="D435i_camera" topics_ns="D435i_camera">
+        <origin xyz="0.05 0 0.3" rpy="0 0 0 " />
+    </xacro:sensor_d435i> -->
     <!-- Variables -->
     <xacro:property name="M_PI" value="3.14159" />
@@ -87,3 +92,41 @@
     <!-- Gazebo definitions  -->
     <xacro:include filename="$(find scout_description)/urdf/scout_v2.gazebo" />
+  <link name="imu_link"/>
+  <joint name="imu_joint" type="fixed">
+    <!-- <origin xyz="0 0 0" rpy="0 ${M_PI} 0" /> -->
+    <origin xyz="0 0 0" rpy="0 0 0" />
+    <parent link="base_link" />
+    <child link="imu_link" />
+  </joint>
+  <xacro:include filename="$(find scout_description)/urdf/camera.xacro" />
+  <xacro:property name="picture_width" value="640" />
+  <xacro:property name="picture_height" value="480" />
+  <xacro:property name="camera_fov" value="${90/180*M_PI}" />
+  <xacro:usb_camera prefix="/camera" parent="base_link" hz="30" fov="${camera_fov}}" width="${picture_width}" height="${picture_height}"
+        x="0.3" y="0.0" z="0.5" roll="0.0" pitch="0.0" yaw="0.0" />
+  <!-- VLP-16 -->
+  <!-- <xacro:include filename="$(find velodyne_description)/urdf/VLP-16.urdf.xacro"/> -->
+  <!-- <xacro:VLP-16 parent="base_link" name="velodyne" topic="/points_raw" hz="10" samples="440" gpu="true" >
+    <origin xyz="0 0 0.6" rpy="0 0 0" />
+  </xacro:VLP-16> -->
+  <!-- imu -->
+  <gazebo reference="imu_link">
+    <gravity>true</gravity>
+    <sensor name="imu_sensor" type="imu">
+      <always_on>true</always_on>
+      <update_rate>200</update_rate>
+      <visualize>true</visualize>
+      <topic>__default_topic__</topic>
+      <plugin filename="libgazebo_ros_imu_sensor.so" name="imu_plugin">
+        <topicName>/imu_raw</topicName>
+        <bodyName>$(arg robot_namespace)/imu_link</bodyName>
+        <updateRateHZ>200.0</updateRateHZ>
+        <gaussianNoise>0.001</gaussianNoise>
+        <xyzOffset>0 0 0</xyzOffset>
+        <rpyOffset>0 0 0</rpyOffset>
+        <frameName>$(arg robot_namespace)/base_link</frameName>
+      </plugin>
+      <pose>0 0 0 0 0 0</pose>
+    </sensor>
+  </gazebo>
 </robot>
